File: VHSBase/VHSBase.kicad_pcb (KiCad board)
At the start: 2 copper layers, 48 x 48 mm, 18 parts, among them J1 Conn_01x03_Female, J10 Conn_01x02_Female, J2 Conn_01x02_Female, J6 Conn_01x07_Female, J7 Conn_01x10_Female, J8 Conn_01x03_Female, J9 Conn_01x02_Female

Commit message: Updated to revision 2.2
Parts:
- removed +5V1, GND1, SCL1, SDA1: Conn_01x03_Female, Pin_Headers:Pin_Header_Straight_1x03_Pitch2.54mm
- removed H3, H4: MountingHole_3.2mm_M3, Mounting_Holes:MountingHole_3.2mm_M3
- added C1: CP, Capacitors_THT:CP_Radial_D5.0mm_P2.00mm, F.Cu at (91.9, 62.2)
- added J11: Conn_01x04_Female, Pin_Headers:Pin_Header_Straight_1x04_Pitch2.54mm, F.Cu at (120.9, 64.2)
- added J12: Conn_01x04_Female, Pin_Headers:Pin_Header_Straight_1x04_Pitch2.54mm, F.Cu at (120.9, 60.5)
- added J3: Conn_01x04_Female, Pin_Headers:Pin_Header_Straight_1x04_Pitch2.54mm, F.Cu at (120.9, 75.1)
- added J4: Conn_01x04_Female, Pin_Headers:Pin_Header_Straight_1x04_Pitch2.54mm, F.Cu at (120.9, 71.5)
- added J5: Conn_01x04_Female, Pin_Headers:Pin_Header_Straight_1x04_Pitch2.54mm, F.Cu at (120.9, 67.8)
- added SRVO1: Conn_01x03_Female, Pin_Headers:Pin_Header_Straight_1x03_Pitch2.54mm, F.Cu at (132.6, 61.9)
- J6: footprint Pin_Headers:Pin_Header_Straight_1x07_Pitch2.54mm -> Pin_Headers:Pin_Header_Straight_1x08_Pitch2.54mm
- moved J9 11.6 mm to (132.6, 74.6), turned to 180 degrees
- moved H1 9.00 mm to (130.9, 93.6)
- moved H2 9.00 mm to (91.0, 93.6)
- moved J10 7.64 mm to (132.6, 82.3), turned to 180 degrees
- moved R1 7.44 mm to (128.5, 80.7), turned to 270 degrees
- moved R2 3.55 mm to (124.5, 80.7), turned to 270 degrees
Connections:
- A1 pad 10: Net-(A1-Pad10) -> /D7
- J7 pad 8: /CS -> /SDCS
Routing:
- net +5V: track 56.0 -> 96.2 mm
- net /COL2: track 37.6 -> 68.5 mm
- net /SDCS: track 0.00 -> 21.6 mm
- net /D7: track 0.00 -> 20.0 mm
- net /SCL: track 16.2 -> 28.5 mm
- net /SDA: track 15.1 -> 27.1 mm
- net /COL1: track 48.1 -> 38.4 mm
- net /COL3: track 46.0 -> 40.6 mm
- net Net-(J10-Pad1): track 4.42 -> 8.74 mm
- net Net-(J9-Pad1): track 4.32 -> 7.74 mm
- net +3V3: track 40.1 -> 43.1 mm
- net /XCS: track 10.9 -> 9.60 mm
Other:
- board text added: "+5v"
- board text added: "Breakout board V2.2 April 2019 Designed by Daniel Oulton For Outside The March"
- board text added: "D7"
- board text added: "SCL"
- board text added: "SDA"
- board text removed: "Breakout board V1.0 March 2019 Designed by Daniel Oulton For Outside The March"
