File: VHSBase/VHSBase.sch (KiCad schematic (older format))
At the start: 14 parts, among them J1 Conn_01x03_Female, J10 Conn_01x02_Female, J2 Conn_01x02_Female, J6 Conn_01x07_Female, J7 Conn_01x10_Female, J8 Conn_01x03_Female, J9 Conn_01x02_Female

Commit message: Updated to revision 2.2
Parts:
- removed +5V1, SCL1, SDA1: Conn_01x03_Female, Pin_Headers:Pin_Header_Straight_1x03_Pitch2.54mm, symbol Connector:Conn_01x03_Female
- added C1: CP, Capacitors_THT:CP_Radial_D5.0mm_P2.00mm, symbol Device:CP
- added J11, J12, J3, J4, J5: Conn_01x04_Female, Pin_Headers:Pin_Header_Straight_1x04_Pitch2.54mm, symbol Connector:Conn_01x04_Female
- added SRVO1: Conn_01x03_Female, Pin_Headers:Pin_Header_Straight_1x03_Pitch2.54mm, symbol Connector:Conn_01x03_Female
- J6: footprint Pin_Headers:Pin_Header_Straight_1x07_Pitch2.54mm -> Pin_Headers:Pin_Header_Straight_1x08_Pitch2.54mm; symbol Connector:Conn_01x07_Female -> Connector:Conn_01x08_Female
Connections:
- net +5V: now also C1.1, J11.2 (Pin_2), J12.2 (Pin_2), J3.2 (Pin_2), J4.2 (Pin_2), J5.2 (Pin_2), SRVO1.2 (Pin_2)
- net COL2: now also SRVO1.3 (Pin_3)
- net GND: now also C1.2, J11.1 (Pin_1), J12.1 (Pin_1), J3.1 (Pin_1), J4.1 (Pin_1), J5.1 (Pin_1), SRVO1.1 (Pin_1)
- net SCL: now also J11.4 (Pin_4), J12.4 (Pin_4), J3.4 (Pin_4), J4.4 (Pin_4), J5.4 (Pin_4)
- net SDA: now also J11.3 (Pin_3), J12.3 (Pin_3), J3.3 (Pin_3), J4.3 (Pin_3), J5.3 (Pin_3)
- net D7: now reaches A1.10 (D7)
- net D7: now also J6.8 (Pin_8)
- no-connect marks 6 -> 5
